File: LED/LED.kicad_pcb (KiCad board)
At the start: 2 copper layers, 42 x 36 mm, 3 parts

Commit message: miniproject1 LED 완성
Parts:
- added SW1: M2011S3A1W03, New_Library_0:Switch_Toggle_SPST_NKK_M2011S3A1x03, F.Cu at (159.2, 83.1)
Connections:
- BT1 pad 1: VCC -> Net-(BT1-+)
Routing:
- net Net-(BT1-+): track 0.00 -> 16.5 mm
- net VCC: track 20.1 -> 21.2 mm, vias 1 -> 0
Other:
- board size 42 x 36 mm -> 55 x 36 mm
Changed lines of the file:
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@@
 		(capping no)
 		(filling no)
-		(zone_defaults)
 		(pcbplotparams
 			(layerselection 0x00000000_00000000_55555555_5755f5ff)
@@
 		)
 	)
+	(footprint "New_Library_0:Switch_Toggle_SPST_NKK_M2011S3A1x03"
+		(layer "F.Cu")
+		(at 159.225 83.075)
+		(property "Reference" "SW1"
+			(at 0 -0.5 0)
+			(unlocked yes)
+			(layer "F.SilkS")
+			(effects
+				(font
+					(size 1 1)
+					(thickness 0.1)
+				)
+			)
+		)
+		(property "Value" "M2011S3A1W03"
+			(at 0 14.1 0)
+			(unlocked yes)
+			(layer "F.Fab")
+			(effects
+				(font
+					(size 1 1)
+					(thickness 0.15)
+				)
+			)
+		)
+		(property "Datasheet" ""
+			(at 0 0 0)
+			(unlocked yes)
+			(layer "F.Fab")
+			(hide yes)
+			(effects
+				(font
+					(size 1 1)
+					(thickness 0.15)
+				)
+			)
+		)
+		(property "Description" ""
+			(at 0 0 0)
+			(unlocked yes)
+			(layer "F.Fab")
+			(hide yes)
+			(effects
+				(font
+					(size 1 1)
+					(thickness 0.15)
+				)
+			)
+		)
+		(sheetname "/")
+		(sheetfile "LED.kicad_sch")
+		(units
+			(unit
+				(name "A")
+				(pins "2" "3")
+			)
+		)
+		(attr through_hole)
+		(duplicate_pad_numbers_are_jumpers no)
+		(fp_rect
+			(start -4.06 -1.91)
+			(end 4.06 11.31)
+			(stroke
+				(width 0.1)
+				(type solid)
+			)
+			(fill no)
+			(layer "F.SilkS")
+		)
+		(fp_rect
+			(start -4.2 -2.05)
+			(end 4.2 11.45)
+			(stroke
+				(width 0.05)
+				(type solid)
+			)
+			(fill no)
+			(layer "F.CrtYd")
+		)
+		(fp_rect
+			(start -3.95 -1.8)
+			(end 3.95 11.2)
+			(stroke
+				(width 0.2)
+				(type solid)
+			)
+			(fill no)
+			(layer "F.Fab")
+		)
+		(fp_text user "${REFERENCE}"
+			(at 0 1.5 0)
+			(unlocked yes)
+			(layer "F.Fab")
+			(effects
+				(font
+					(size 1 1)
+					(thickness 0.15)
+				)
+			)
+		)
+		(pad "2" thru_hole circle
+			(at 0 4.7)
+			(size 2.22 2.22)
+			(drill 1.62)
+			(layers "*.Cu" "*.Mask")
+			(remove_unused_layers no)
+			(net "Net-(BT1-+)")
+			(pinfunction "A_2")
+			(pintype "passive")
+		)
+		(pad "3" thru_hole circle
+			(at 0 9.4)
+			(size 2.22 2.22)
+			(drill 1.62)
+			(layers "*.Cu" "*.Mask")
+			(remove_unused_layers no)
+			(net "VCC")
+			(pinfunction "A_3")
+			(pintype "passive")
+		)
+		(embedded_fonts no)
+	)
 	(footprint "Battery:BatteryHolder_Keystone_1058_1x2032"
 		(layer "B.Cu")
@@
 			(size 2.54 3.51)
 			(layers "B.Cu" "B.Mask" "B.Paste")
-			(net "VCC")
+			(net "Net-(BT1-+)")
 			(pinfunction "+_1")
 			(pintype "passive")
@@
 	(gr_rect
 		(start 110 70)
-		(end 152 106)
+		(end 165 106)
 		(stroke
 			(width 0.05)
@@
 	)
 	(segment
-		(start 144 100)
-		(end 142 102)
+		(start 116 102)
+		(end 139.46 102)
 		(width 0.2)
 		(layer "F.Cu")
-		(net "VCC")
+		(net "/ex.led")
 	)
 	(segment
-		(start 144 93)
-		(end 144 100)
+		(start 116 102.35)
+		(end 116 102)
 		(width 0.2)
 		(layer "F.Cu")
-		(net "VCC")
-	)
-	(via
-		(at 144 93)
-		(size 0.6)
-		(drill 0.3)
-		(layers "F.Cu" "B.Cu")
-		(net "VCC")
-	)
-	(segment
-		(start 144.68 83)
-		(end 144.68 92.32)
-		(width 0.2)
-		(layer "B.Cu")
-		(net "VCC")
-	)
-	(segment
-		(start 144.68 92.32)
-		(end 144 93)
-		(width 0.2)
-		(layer "B.Cu")
-		(net "VCC")
+		(net "/ex.led")
 	)
 	(segment
@@
 	)
 	(segment
-		(start 116 102)
-		(end 139.46 102)
+		(start 142 102)
+		(end 149.7 102)
 		(width 0.2)
 		(layer "F.Cu")
-		(net "/ex.led")
+		(net "VCC")
 	)
 	(segment
-		(start 116 102.35)
-		(end 116 102)
+		(start 149.7 102)
+		(end 159.225 92.475)
 		(width 0.2)
 		(layer "F.Cu")
-		(net "/ex.led")
+		(net "VCC")
+	)
+	(segment
+		(start 154.45 83)
+		(end 144.68 83)
+		(width 0.2)
+		(layer "B.Cu")
+		(net "Net-(BT1-+)")
+	)
+	(segment
+		(start 159.225 87.775)
+		(end 154.45 83)
+		(width 0.2)
+		(layer "B.Cu")
+		(net "Net-(BT1-+)")
 	)
 	(zone
@@
 		(polygon
 			(pts
-				(xy 110 70) (xy 110 106) (xy 152 106) (xy 152 70)
-			)
-		)
+				(xy 110 70) (xy 110 106) (xy 165 106) (xy 165 70)
+			)
+		)
