File: LED/LED.kicad_sch (KiCad schematic)
At the start: 3 parts

Commit message: miniproject1 LED 완성
Parts:
- added SW1: M2011S3A1W03, New_Library_0:Switch_Toggle_SPST_NKK_M2011S3A1x03, symbol New_Library_0:M2011S3A1W03
Connections:
- net VCC: now also SW1.3 (A); no longer BT1.1 (+)
- new net: BT1.1 (+), SW1.2 (A)
Other:
- moved on the sheet: BT1
Changed lines of the file:
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@@
-	)
-	(junction
-		(at 114.3 92.71)
-		(diameter 0)
-		(color 0 0 0 0)
 	)
 	(junction
@@
 	)
 	(junction
-		(at 93.98 63.5)
+		(at 114.3 99.06)
 		(diameter 0)
 		(color 0 0 0 0)
@@
 		(color 0 0 0 0)
 	)
+	(junction
+		(at 93.98 63.5)
+		(diameter 0)
+		(color 0 0 0 0)
+	)
 	(wire
 		(pts
@@
 	(wire
 		(pts
-			(xy 114.3 101.6) (xy 114.3 92.71)
+			(xy 114.3 95.25) (xy 114.3 99.06)
+		)
+		(stroke
+			(width 0)
+			(type default)
+		)
+	)
+	(wire
+		(pts
+			(xy 114.3 101.6) (xy 114.3 99.06)
 		)
 		(stroke
@@
 	(wire
 		(pts
-			(xy 114.3 92.71) (xy 114.3 81.28)
-		)
-		(stroke
-			(width 0)
-			(type default)
-		)
-	)
-	(wire
-		(pts
 			(xy 78.74 101.6) (xy 78.74 97.79)
 		)
@@
 	(wire
 		(pts
+			(xy 114.3 87.63) (xy 114.3 83.82)
+		)
+		(stroke
+			(width 0)
+			(type default)
+		)
+	)
+	(wire
+		(pts
+			(xy 78.74 101.6) (xy 95.25 101.6)
+		)
+		(stroke
+			(width 0)
+			(type default)
+		)
+	)
+	(wire
+		(pts
+			(xy 78.74 63.5) (xy 78.74 67.31)
+		)
+		(stroke
+			(width 0)
+			(type default)
+		)
+	)
+	(wire
+		(pts
 			(xy 114.3 73.66) (xy 114.3 67.31)
-		)
-		(stroke
-			(width 0)
-			(type default)
-		)
-	)
-	(wire
-		(pts
-			(xy 78.74 101.6) (xy 95.25 101.6)
-		)
-		(stroke
-			(width 0)
-			(type default)
-		)
-	)
-	(wire
-		(pts
-			(xy 78.74 63.5) (xy 78.74 67.31)
 		)
 		(stroke
@@
 	(symbol
 		(lib_id "Device:Battery_Cell")
-		(at 114.3 78.74 0)
+		(at 114.3 92.71 0)
 		(unit 1)
 		(body_style 1)
@@
 		(fields_autoplaced yes)
 		(property "Reference" "BT1"
-			(at 118.11 75.6284 0)
+			(at 118.11 89.5984 0)
 			(show_name no)
 			(do_not_autoplace no)
@@
 		)
 		(property "Value" "3V"
-			(at 118.11 78.1684 0)
+			(at 118.11 92.1384 0)
 			(show_name no)
 			(do_not_autoplace no)
@@
 		)
 		(property "Footprint" "Battery:BatteryHolder_Keystone_1058_1x2032"
-			(at 114.3 77.216 90)
+			(at 114.3 91.186 90)
 			(hide yes)
 			(show_name no)
@@
 		)
 		(property "Datasheet" ""
-			(at 114.3 77.216 90)
+			(at 114.3 91.186 90)
 			(hide yes)
 			(show_name no)
@@
 		)
 		(property "Description" "Single-cell battery"
-			(at 114.3 78.74 0)
+			(at 114.3 92.71 0)
 			(hide yes)
 			(show_name no)
@@
 		)
 		(property "Sim.Device" "V"
-			(at 114.3 78.74 0)
+			(at 114.3 92.71 0)
 			(hide yes)
 			(show_name no)
@@
 		)
 		(property "Sim.Type" "DC"
-			(at 114.3 78.74 0)
+			(at 114.3 92.71 0)
 			(hide yes)
 			(show_name no)
@@
 		)
 		(property "Sim.Pins" "1=+ 2=-"
-			(at 114.3 78.74 0)
+			(at 114.3 92.71 0)
 			(hide yes)
 			(show_name no)
@@
 	)
 	(symbol
+		(lib_id "New_Library_0:M2011S3A1W03")
+		(at 114.3 78.74 90)
+		(unit 1)
+		(body_style 1)
+		(exclude_from_sim no)
+		(in_bom yes)
+		(on_board yes)
+		(in_pos_files yes)
+		(dnp no)
+		(fields_autoplaced yes)
+		(property "Reference" "SW1"
+			(at 115.57 77.4699 90)
+			(show_name no)
+			(do_not_autoplace no)
+			(effects
+				(font
+					(size 1.27 1.27)
+				)
+				(justify right)
+			)
+		)
+		(property "Value" "M2011S3A1W03"
+			(at 115.57 80.0099 90)
+			(show_name no)
+			(do_not_autoplace no)
+			(effects
+				(font
+					(size 1.27 1.27)
+				)
+				(justify right)
+			)
+		)
+		(property "Footprint" "New_Library_0:Switch_Toggle_SPST_NKK_M2011S3A1x03"
+			(at 114.3 78.74 0)
+			(hide yes)
+			(show_name no)
+			(do_not_autoplace no)
+			(effects
+				(font
+					(size 1.27 1.27)
+				)
+			)
+		)
+		(property "Datasheet" ""
+			(at 114.3 78.74 0)
+			(hide yes)
+			(show_name no)
+			(do_not_autoplace no)
+			(effects
+				(font
+					(size 1.27 1.27)
+				)
+			)
+		)
+		(property "Description" ""
+			(at 114.3 78.74 0)
+			(hide yes)
+			(show_name no)
+			(do_not_autoplace no)
+			(effects
+				(font
+					(size 1.27 1.27)
+				)
+			)
+		)
+		(pin "2"
+		)
+		(pin "3"
+		)
+		(instances
+			(project "LED"
+				(path "/37335d2c-2aea-4f24-9a80-082e17e2082f"
+					(reference "SW1")
+					(unit 1)
+				)
+			)
+		)
+	)
+	(symbol
 		(lib_id "power:PWR_FLAG")
 		(at 114.3 67.31 270)
@@
 	(symbol
 		(lib_id "power:PWR_FLAG")
-		(at 114.3 92.71 270)
+		(at 114.3 99.06 270)
 		(unit 1)
 		(body_style 1)
@@
 		(fields_autoplaced yes)
 		(property "Reference" "#FLG02"
-			(at 116.205 92.71 0)
+			(at 116.205 99.06 0)
 			(hide yes)
 			(show_name no)
@@
 		)
 		(property "Value" "PWR_FLAG"
-			(at 118.11 92.7099 90)
+			(at 118.11 99.0599 90)
 			(show_name no)
 			(do_not_autoplace no)
@@
 		)
 		(property "Footprint" ""
-			(at 114.3 92.71 0)
+			(at 114.3 99.06 0)
 			(hide yes)
 			(show_name no)
@@
 		)
 		(property "Datasheet" ""
-			(at 114.3 92.71 0)
+			(at 114.3 99.06 0)
 			(hide yes)
 			(show_name no)
@@
 		)
 		(property "Description" "Special symbol for telling ERC where power comes from"
-			(at 114.3 92.71 0)
-			(hide yes)
-			(show_name no)
+			(at 114.3 99.06 0)
+			(hide yes)
+			(show_name no)
