File: getting-started/getting-started.kicad_pcb (KiCad board)
At the start: 2 copper layers, 45 x 36 mm, 3 parts

Commit message: update
Parts:
- added SW1: M2011S3A1W03, getting-started:Switch_Toggle_SPST_NKK_M2011S3A1x03, F.Cu at (163.0, 75.8)
Connections:
- BT1 pad 1: VCC -> Net-(BT1-+)
Routing:
- net Net-(BT1-+): track 0.00 -> 12.7 mm
- net VCC: track 15.5 -> 11.0 mm, vias 1 -> 0
Other:
- board size 45 x 36 mm -> 52.5 x 36 mm
Changed lines of the file:
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@@
 		)
+	)
+	(footprint "getting-started:Switch_Toggle_SPST_NKK_M2011S3A1x03"
+		(layer "F.Cu")
+		(at 163 75.8)
+		(property "Reference" "SW1"
+			(at 0 -0.5 0)
+			(unlocked yes)
+			(layer "F.SilkS")
+			(effects
+				(font
+					(size 1 1)
+					(thickness 0.1)
+				)
+			)
+		)
+		(property "Value" "M2011S3A1W03"
+			(at 0 1 0)
+			(unlocked yes)
+			(layer "F.Fab")
+			(effects
+				(font
+					(size 1 1)
+					(thickness 0.15)
+				)
+			)
+		)
+		(property "Datasheet" ""
+			(at 0 0 0)
+			(unlocked yes)
+			(layer "F.Fab")
+			(hide yes)
+			(effects
+				(font
+					(size 1 1)
+					(thickness 0.15)
+				)
+			)
+		)
+		(property "Description" ""
+			(at 0 0 0)
+			(unlocked yes)
+			(layer "F.Fab")
+			(hide yes)
+			(effects
+				(font
+					(size 1 1)
+					(thickness 0.15)
+				)
+			)
+		)
+		(sheetname "/")
+		(sheetfile "getting-started.kicad_sch")
+		(units
+			(unit
+				(name "A")
+				(pins "2" "3")
+			)
+		)
+		(attr through_hole)
+		(duplicate_pad_numbers_are_jumpers no)
+		(fp_rect
+			(start -4.06 -1.91)
+			(end 4.06 11.31)
+			(stroke
+				(width 0.12)
+				(type solid)
+			)
+			(fill no)
+			(layer "F.SilkS")
+		)
+		(fp_rect
+			(start -4.2 -2.05)
+			(end 4.2 11.45)
+			(stroke
+				(width 0.05)
+				(type solid)
+			)
+			(fill no)
+			(layer "F.CrtYd")
+		)
+		(fp_rect
+			(start -3.95 -1.8)
+			(end 3.95 11.2)
+			(stroke
+				(width 0.1)
+				(type solid)
+			)
+			(fill no)
+			(layer "F.Fab")
+		)
+		(fp_text user "${REFERENCE}"
+			(at 0 2.5 0)
+			(unlocked yes)
+			(layer "F.Fab")
+			(effects
+				(font
+					(size 1 1)
+					(thickness 0.15)
+				)
+			)
+		)
+		(pad "2" thru_hole circle
+			(at 0 4.7)
+			(size 2.22 2.22)
+			(drill 1.62)
+			(layers "*.Cu" "*.Mask")
+			(remove_unused_layers no)
+			(net "Net-(BT1-+)")
+			(pinfunction "A_2")
+			(pintype "passive")
+		)
+		(pad "3" thru_hole circle
+			(at 0 9.4)
+			(size 2.22 2.22)
+			(drill 1.62)
+			(layers "*.Cu" "*.Mask")
+			(remove_unused_layers no)
+			(net "VCC")
+			(pinfunction "B_3")
+			(pintype "passive")
+		)
+		(embedded_fonts no)
 	)
 	(footprint "LED_THT:LED_D5.0mm"
@@
 			(size 2.54 3.51)
 			(layers "B.Cu" "B.Mask" "B.Paste")
-			(net "VCC")
+			(net "Net-(BT1-+)")
 			(pinfunction "+_1")
 			(pintype "passive")
@@
 	(gr_rect
 		(start 117 61)
-		(end 162 97)
+		(end 169.5 97)
 		(stroke
 			(width 0.05)
@@
 	)
 	(segment
-		(start 154 90)
-		(end 154.35 89.65)
+		(start 158.2 90)
+		(end 163 85.2)
 		(width 0.4)
 		(layer "F.Cu")
@@
 	)
 	(segment
-		(start 154.35 83.35)
-		(end 154 83)
+		(start 154 90)
+		(end 158.2 90)
 		(width 0.4)
 		(layer "F.Cu")
-		(net "VCC")
-	)
-	(segment
-		(start 154.35 89.65)
-		(end 154.35 83.35)
-		(width 0.4)
-		(layer "F.Cu")
-		(net "VCC")
-	)
-	(via
-		(at 154 83)
-		(size 0.6)
-		(drill 0.3)
-		(layers "F.Cu" "B.Cu")
-		(net "VCC")
-	)
-	(segment
-		(start 154 83)
-		(end 154.155 82.845)
-		(width 0.4)
-		(layer "B.Cu")
-		(net "VCC")
-	)
-	(segment
-		(start 154.155 82.845)
-		(end 154.155 74.82397)
-		(width 0.4)
-		(layer "B.Cu")
 		(net "VCC")
 	)
@@
 		(net "GND")
 	)
+	(segment
+		(start 163 78)
+		(end 159.82397 74.82397)
+		(width 0.4)
+		(layer "B.Cu")
+		(net "Net-(BT1-+)")
+	)
+	(segment
+		(start 163 80.5)
+		(end 163 78)
+		(width 0.4)
+		(layer "B.Cu")
+		(net "Net-(BT1-+)")
+	)
+	(segment
+		(start 159.82397 74.82397)
+		(end 154.155 74.82397)
+		(width 0.4)
+		(layer "B.Cu")
+		(net "Net-(BT1-+)")
+	)
 	(zone
 		(net "GND")
@@
 		(polygon
 			(pts
-				(xy 117 61) (xy 117 97) (xy 162 97) (xy 162 61)
-			)
-		)
+				(xy 117 61) (xy 117 97) (xy 169.5 97) (xy 169.5 61)
+			)
+		)
