File: getting-started/getting-started.kicad_sch (KiCad schematic)
At the start: 4 parts, among them SW1 M2011S3A1W03

Commit message: 1
Parts:
- removed BT1: 3V, Battery:BatteryHolder_Keystone_1058_1x2032, symbol Device:Battery_Cell
- removed SW1: M2011S3A1W03, New_Library_0:Switch_Toggle_SPST_NKK_M2011S3A1x03, symbol New_Library_0:M2011S3A1W03
- added BT1: 3V, Battery:BatteryHolder_Keystone_1058_1x2032, symbol Device:Battery
Connections:
- net GND: now also D1.1 (K), BT1.2 (-); no longer R1.2
- net VCC: now also R1.1, BT1.1 (+); no longer D1.2 (A)
- removed net ex.led: D1.1 (K), R1.1
- new net led: D1.2 (A), R1.2
Other:
- title: Led Blank in KiCad 10.0 -> getting-started

Commit message: update
Parts:
- added SW1: M2011S3A1W03, getting-started:Switch_Toggle_SPST_NKK_M2011S3A1x03, symbol getting-started:M2011S3A1W03
Connections:
- net VCC: now also SW1.3 (B); no longer BT1.1 (+)
- new net: BT1.1 (+), SW1.2 (A)
Other:
- moved on the sheet: BT1
Changed lines of the file:
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@@
+	)
+	(junction
+		(at 185.42 139.7)
+		(diameter 0)
+		(color 0 0 0 0)
 	)
 	(junction
@@
 		(color 0 0 0 0)
 	)
-	(junction
-		(at 185.42 139.7)
-		(diameter 0)
-		(color 0 0 0 0)
-	)
-	(wire
-		(pts
-			(xy 185.42 128.27) (xy 185.42 139.7)
-		)
-		(stroke
-			(width 0)
-			(type default)
-		)
-	)
-	(wire
-		(pts
-			(xy 185.42 109.22) (xy 185.42 118.11)
+	(wire
+		(pts
+			(xy 185.42 135.89) (xy 185.42 139.7)
+		)
+		(stroke
+			(width 0)
+			(type default)
+		)
+	)
+	(wire
+		(pts
+			(xy 185.42 109.22) (xy 185.42 111.76)
 		)
 		(stroke
@@
 		(pts
 			(xy 185.42 139.7) (xy 185.42 144.78)
+		)
+		(stroke
+			(width 0)
+			(type default)
+		)
+	)
+	(wire
+		(pts
+			(xy 185.42 121.92) (xy 185.42 125.73)
 		)
 		(stroke
@@
 			)
 			(justify right bottom)
+		)
+	)
+	(symbol
+		(lib_id "getting-started:M2011S3A1W03")
+		(at 185.42 116.84 90)
+		(unit 1)
+		(body_style 1)
+		(exclude_from_sim no)
+		(in_bom yes)
+		(on_board yes)
+		(in_pos_files yes)
+		(dnp no)
+		(fields_autoplaced yes)
+		(property "Reference" "SW1"
+			(at 186.69 115.5699 90)
+			(show_name no)
+			(do_not_autoplace no)
+			(effects
+				(font
+					(size 1.27 1.27)
+				)
+				(justify right)
+			)
+		)
+		(property "Value" "M2011S3A1W03"
+			(at 186.69 118.1099 90)
+			(show_name no)
+			(do_not_autoplace no)
+			(effects
+				(font
+					(size 1.27 1.27)
+				)
+				(justify right)
+			)
+		)
+		(property "Footprint" "getting-started:Switch_Toggle_SPST_NKK_M2011S3A1x03"
+			(at 185.42 116.84 0)
+			(hide yes)
+			(show_name no)
+			(do_not_autoplace no)
+			(effects
+				(font
+					(size 1.27 1.27)
+				)
+			)
+		)
+		(property "Datasheet" ""
+			(at 185.42 116.84 0)
+			(hide yes)
+			(show_name no)
+			(do_not_autoplace no)
+			(effects
+				(font
+					(size 1.27 1.27)
+				)
+			)
+		)
+		(property "Description" ""
+			(at 185.42 116.84 0)
+			(hide yes)
+			(show_name no)
+			(do_not_autoplace no)
+			(effects
+				(font
+					(size 1.27 1.27)
+				)
+			)
+		)
+		(pin "2"
+		)
+		(pin "3"
+		)
+		(instances
+			(project "getting-started"
+				(path "/87f57f61-2932-4fe4-97d6-165a3b3b1dee"
+					(reference "SW1")
+					(unit 1)
+				)
+			)
 		)
 	)
@@
 	(symbol
 		(lib_id "Device:Battery")
-		(at 185.42 123.19 0)
+		(at 185.42 130.81 0)
 		(unit 1)
 		(body_style 1)
@@
 		(fields_autoplaced yes)
 		(property "Reference" "BT1"
-			(at 189.23 121.3484 0)
+			(at 189.23 128.9684 0)
 			(show_name no)
 			(do_not_autoplace no)
@@
 		)
 		(property "Value" "3V"
-			(at 189.23 123.8884 0)
+			(at 189.23 131.5084 0)
 			(show_name no)
 			(do_not_autoplace no)
@@
 		)
 		(property "Footprint" "Battery:BatteryHolder_Keystone_1058_1x2032"
-			(at 185.42 121.666 90)
+			(at 185.42 129.286 90)
 			(hide yes)
 			(show_name no)
@@
 		)
 		(property "Datasheet" ""
-			(at 185.42 121.666 90)
+			(at 185.42 129.286 90)
 			(hide yes)
 			(show_name no)
@@
 		)
 		(property "Description" "Multiple-cell battery"
-			(at 185.42 123.19 0)
+			(at 185.42 130.81 0)
 			(hide yes)
 			(show_name no)
@@
 		)
 		(property "Sim.Device" "V"
-			(at 185.42 123.19 0)
+			(at 185.42 130.81 0)
 			(hide yes)
 			(show_name no)
@@
 		)
 		(property "Sim.Type" "DC"
-			(at 185.42 123.19 0)
+			(at 185.42 130.81 0)
 			(hide yes)
 			(show_name no)
@@
 		)
 		(property "Sim.Pins" "1=+ 2=-"
-			(at 185.42 123.19 0)
-			(hide yes)
-			(show_name no)
+			(at 185.42 130.81 0)
+			(hide yes)
+			(show_name no)
