File: ArduinoNano/ArduinoNano.kicad_sch (KiCad schematic)
At the start: 15 parts, among them SW1 RESET, U1 ATmega328P-A, U2 FT232RL, Y1 16MHz

Commit message: update
Parts:
- added C2: 4.7uF _16V, Capacitor_Tantalum_SMD:CP_EIA-3216-18_Kemet-A, symbol Device:C_Polarized
- added C8: 1uF, Capacitor_SMD:C_0603_1608Metric, symbol Device:C
- added C9: 100nF, Capacitor_SMD:C_0603_1608Metric, symbol Device:C
- added D1: SS1P3L, Diode_SMD:D_SMP_DO-220AA, symbol Device:D_Schottky
- added F1: MF-MSMF050-2 500mA, Fuse:Fuse_0603_1608Metric, symbol Device:Polyfuse
- added IC2: LM1117MP-5.0, Package_TO_SOT_SMD:SOT-223, symbol Regulator_Linear:LM1117MP-5.0
- added J1, J2: XXXX_STRIPNANO, Connector_PinHeader_2.54mm:PinHeader_1x15_P2.54mm_Vertical, symbol Connector:Conn_01x15_Pin
- added J3: USB_B_Mini, Connector_USB:USB_Mini-B_Wuerth_65100516121_Horizontal, symbol Connector:USB_B_Mini
- added J4: ICSP, Connector_PinHeader_2.54mm:PinHeader_2x03_P2.54mm_Vertical, symbol Connector_Generic:Conn_02x03_Odd_Even
- added PWR1: Green, LED_SMD:LED_0805_2012Metric, symbol Device:LED
- C1, C3, C4, C6, C7: footprint (none) -> Capacitor_SMD:C_0603_1608Metric
- C5: footprint (none) -> Capacitor_Tantalum_SMD:CP_EIA-1608-08_AVX-J
- IC3: renamed from U1; footprint Package_QFP:TQFP-32_7x7mm_P0.8mm -> Package_DFN_QFN:VQFN-32-1EP_5x5mm_P0.5mm_EP3.1x3.1mm
- L1, RX1, TX1: footprint (none) -> LED_SMD:LED_0805_2012Metric
- RN1, RN2: footprint (none) -> Resistor_SMD:R_Array_Concave_4x0603
- SWe1: renamed from SW1; footprint Button_Switch_THT:SW_PUSH_6mm -> Button_Switch_SMD:SW_Push_1P1T_NO_CK_KMR2
- Y1: footprint (none) -> Crystal:Resonator_SMD_Murata_CSTxExxV-3Pin_3.0x1.1mm
- renumbered U2 to IC1
Connections:
- net +5V: now also C8.1, D1.1 (K), J2.4 (Pin_4), J4.2 (Pin_2); no longer C6.1, IC1.17 (3V3OUT)
- net A0: now also J2.12 (Pin_12)
- net A1: now also J2.11 (Pin_11)
- net A2: now also J2.10 (Pin_10)
- net A3: now also J2.9 (Pin_9)
- net A4: now also J2.8 (Pin_8)
- net A5: now also J2.7 (Pin_7)
- net A6: now also J2.6 (Pin_6)
- net A7: now also J2.5 (Pin_5)
- net AREF: now also J2.13 (Pin_13)
- net D0/RX: now also J1.2 (Pin_2)
- net D10: now also J1.13 (Pin_13)
- net D11/MOSI: now also J1.14 (Pin_14), J4.4 (Pin_4)
- net D12/MISO: now also J1.15 (Pin_15), J4.1 (Pin_1)
- net D13/SCK: now also J2.15 (Pin_15), J4.3 (Pin_3)
- net D1/TX: now also J1.1 (Pin_1)
- net D2: now also J1.5 (Pin_5)
- net D3: now also J1.6 (Pin_6)
- net D4: now also J1.7 (Pin_7)
- net D5: now also J1.8 (Pin_8)
- net D6: now also J1.9 (Pin_9)
- net D7: now also J1.10 (Pin_10)
- net D8: now also J1.11 (Pin_11)
- net D9: now also J1.12 (Pin_12)
- net GND: now also C2.2, C8.2, C9.2, IC2.1 (GND), J1.4 (Pin_4), J2.2 (Pin_2), J3.5 (GND), J3.SH (Shield), J4.6 (Pin_6), PWR1.1 (K)
- net RESET: now also J1.3 (Pin_3), J2.3 (Pin_3), J4.5 (Pin_5)
- net at RN1.3 (R3.1): now also PWR1.2 (A)
- net at RN1.6 (R3.2): now also IC2.2 (VO)
- net at IC1.15 (USBD+): now also J3.3 (D+)
- net at IC1.16 (USBD-): now also J3.2 (D-)
- new net: F1.2, J3.1 (VBUS)
- new net +3V3: C6.1, IC1.17 (3V3OUT), J2.14 (Pin_14)
- new net VIN: IC2.3 (VI), J2.1 (Pin_1)
- new net VUSB: C2.1, C9.1, D1.2 (A), F1.1
- no-connect marks 0 -> 12
Other:
- note added: "+5V AUTO SELECTOR"
- note added: "+5V REG"
- note added: "ICSP"
- note added: "USB"
- moved on the sheet: C1, C3, C4, C5, C6, C7, IC1, IC3, L1, RN1A, RN1B, RN1C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

Commit message: update
Connections:
- no-connect marks 12 -> 34
Changed lines of the file:
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@@
+	)
+	(no_connect
+		(at 240.03 163.83)
 	)
 	(no_connect
@@
 	)
 	(no_connect
+		(at 227.33 162.56)
+	)
+	(no_connect
+		(at 232.41 162.56)
+	)
+	(no_connect
+		(at 234.95 163.83)
+	)
+	(no_connect
 		(at 289.56 138.43)
+	)
+	(no_connect
+		(at 237.49 161.29)
 	)
 	(no_connect
@@
 	)
 	(no_connect
+		(at 234.95 168.91)
+	)
+	(no_connect
+		(at 238.76 161.29)
+	)
+	(no_connect
+		(at 240.03 161.29)
+	)
+	(no_connect
 		(at 289.56 125.73)
+	)
+	(no_connect
+		(at 231.14 161.29)
+	)
+	(no_connect
+		(at 237.49 166.37)
 	)
 	(no_connect
@@
 	)
 	(no_connect
+		(at 233.68 168.91)
+	)
+	(no_connect
 		(at 248.92 125.73)
+	)
+	(no_connect
+		(at 233.68 163.83)
+	)
+	(no_connect
+		(at 232.41 167.64)
 	)
 	(no_connect
@@
 	)
 	(no_connect
+		(at 228.6 163.83)
+	)
+	(no_connect
+		(at 236.22 162.56)
+	)
+	(no_connect
+		(at 229.87 165.1)
+	)
+	(no_connect
 		(at 289.56 115.57)
+	)
+	(no_connect
+		(at 228.6 161.29)
+	)
+	(no_connect
+		(at 241.3 162.56)
+	)
+	(no_connect
+		(at 236.22 167.64)
+	)
+	(no_connect
+		(at 229.87 161.29)
 	)
 	(no_connect
@@
 	)
 	(no_connect
+		(at 231.14 166.37)
+	)
+	(no_connect
+		(at 238.76 165.1)
+	)
+	(no_connect
